File: amp.kicad_sch (KiCad schematic)
At the start: 11 parts, among them IC301 MAX98357AETE+T, IC302 MAX98357AETE+T, J301 L_SPKR, J302 R_SPKR

Commit message: updated to rev 3
Parts:
- removed C21, C26: 10u, Capacitor_SMD:C_0603_1608Metric, symbol Device:C_Small
- added C303, C307: 10u, Capacitor_SMD:C_0805_2012Metric, symbol Device:C_Polarized_Small
- added JP301, JP305: GAIN, Jumper:SolderJumper-3_P1.3mm_Open_RoundedPad1.0x1.5mm, symbol Jumper:Jumper_3_Open
- added R302: 0, Resistor_SMD:R_0603_1608Metric, symbol Device:R_Small
- C301: renamed from C23; footprint Capacitor_SMD:C_0402_1005Metric -> Capacitor_SMD:C_0603_1608Metric
- C302: renamed from C22; footprint Capacitor_SMD:C_0402_1005Metric -> Capacitor_SMD:C_0603_1608Metric
- C304: renamed from C24; footprint Capacitor_SMD:C_0402_1005Metric -> Capacitor_SMD:C_0603_1608Metric
- C305: renamed from C25; footprint Capacitor_SMD:C_0402_1005Metric -> Capacitor_SMD:C_0603_1608Metric
- R301: renamed from R15; footprint Resistor_SMD:R_0402_1005Metric -> Resistor_SMD:R_0603_1608Metric
Connections:
- net +5V: now also C303.1, C307.1, JP301.1 (A), JP305.1 (A); no longer IC301.2 (GAIN), IC301.4 (~{SD_MODE}), IC302.2 (GAIN), R301.1
- net GND: now also C303.2, C307.2, JP301.3 (B), JP305.3 (B)
- net I2SO_BCK_OUT renamed I2S0_BCK_IN
- net I2SO_SD_OUT renamed I2S0_SD_IN
- net I2SO_WS_OUT renamed I2S0_WS_IN
- new net: IC301.2 (GAIN), JP305.2 (C)
- new net: IC301.4 (~{SD_MODE}), R302.2
- new net: IC302.2 (GAIN), JP301.2 (C)
- new net AMP_SW: R301.1, R302.1
Other:
- note added: "DEFAULT GAIN: 9dB"

Commit message: updated to rev 4
Parts:
- added R303, R304: 100k, Resistor_SMD:R_0402_1005Metric, symbol Device:R_Small
- C301, C302, C304, C305: footprint Capacitor_SMD:C_0603_1608Metric -> Capacitor_SMD:C_0402_1005Metric; JLCPCB Part # (none) -> C1525; LCSC C1525 -> (none)
- C303, C307: footprint Capacitor_SMD:C_0805_2012Metric -> Capacitor_SMD:C_0603_1608Metric; JLCPCB Part # (none) -> C96446
- IC301, IC302: JLCPCB Part # (none) -> C910544; LCSC C910544 -> (none)
- R301: footprint Resistor_SMD:R_0603_1608Metric -> Resistor_SMD:R_0402_1005Metric; JLCPCB Part # (none) -> C45956; LCSC C45956 -> (none)
- R302: footprint Resistor_SMD:R_0603_1608Metric -> Resistor_SMD:R_0402_1005Metric; JLCPCB Part # (none) -> C17168; LCSC C45956 -> (none)
Connections:
- net GND: now also R303.2, R304.2
- net at IC301.4 (~{SD_MODE}), R302.2: now also R303.1
- net at IC302.4 (~{SD_MODE}), R301.2: now also R304.1
Other:
- moved on the sheet: C301, C302, C303, C304, C305, C307, IC301, IC302, J301, JP301, JP305, R302
